Commit message: Add Elliptical path trace

File: Stewart/Stewart.urdf (robot description, URDF)
Before this commit: robot Stewart, 51 links, 50 joints
Joints:
- joint Revolute_10: axis 0.841524 -0.485854 0.236183 -> 0.841174 -0.485652 0.23784; origin xyz=0.034419 0.009573 0.006081 rpy=0 0 0 -> xyz=0.03441 0.009579 0.006124 rpy=0 0 0
- joint Revolute_11: axis 0.779901 0.450276 0.434747 -> 0.780387 0.450557 0.433584; origin xyz=0.007332 0.033679 0.011194 rpy=0 0 0 -> xyz=0.007345 0.033686 0.011164 rpy=0 0 0
- joint Revolute_12: axis 0.842492 0.486413 -0.231539 -> 0.842824 0.486605 -0.229918; origin xyz=0.008944 0.034609 -0.005963 rpy=0 0 0 -> xyz=0.008953 0.034614 -0.005921 rpy=0 0 0
- joint Revolute_19: axis 0.371624 -0.217029 0.902659 -> 0.369151 -0.214507 0.904276; origin xyz=0.0 0.0 0.0 rpy=0 0 0 -> xyz=0.000223 -0.000129 0.000545 rpy=0 0 0
- joint Revolute_20: axis -0.002141 0.434195 0.900816 -> -0.00375 0.434573 0.900629; origin xyz=0.0 0.0 0.0 rpy=0 0 0 -> xyz=-4e-06 0.00048 0.000995 rpy=0 0 0
- joint Revolute_21: axis -0.377094 -0.216348 0.900552 -> -0.377381 -0.213518 0.901107; origin xyz=0.0 0.0 0.0 rpy=0 0 0 -> xyz=-0.000369 -0.00021 0.000883 rpy=0 0 0
- joint Revolute_22: axis -0.379236 -0.217587 0.899353 -> -0.379485 -0.214736 0.899933; origin xyz=0.0 0.0 1e-06 rpy=0 0 0 -> xyz=-0.000399 -0.000226 0.000946 rpy=0 0 0
- joint Revolute_23: axis -0.002144 0.431721 0.902005 -> -0.003749 0.431354 0.902175; origin xyz=0.0 1e-06 0.0 rpy=0 0 0 -> xyz=-6e-06 0.000667 0.001393 rpy=0 0 0
- joint Revolute_24: axis 0.373767 -0.218269 0.901475 -> 0.370839 -0.215482 0.903353; origin xyz=0.0 0.0 0.0 rpy=0 0 0 -> xyz=0.00037 -0.000214 0.0009 rpy=0 0 0
- joint Revolute_25: axis -0.7793 -0.448919 -0.437223 -> -0.779795 -0.449231 -0.436018; origin xyz=0.004701 0.002742 0.047128 rpy=0 0 0 -> xyz=0.004703 0.002865 0.047121 rpy=0 0 0
- joint Revolute_26: axis -0.843721 -0.484609 0.230843 -> -0.844029 -0.484671 0.229586; origin xyz=0.036382 0.003675 0.030225 rpy=0 0 0 -> xyz=0.036291 0.003778 0.030321 rpy=0 0 0
- joint Revolute_27: axis -0.779688 0.452487 0.43283 -> -0.78153 0.453054 0.428898; origin xyz=0.034835 -0.02027 0.025026 rpy=0 0 0 -> xyz=0.034764 -0.020174 0.025202 rpy=0 0 0
- joint Revolute_28: axis -0.840937 0.487325 -0.235244 -> -0.840501 0.487444 -0.236553; origin xyz=0.021358 0.004844 0.042084 rpy=0 0 0 -> xyz=0.021283 0.004826 0.042124 rpy=0 0 0
- joint Revolute_29: axis 0.49842 -0.866934 0.001748 -> 0.498367 -0.866964 0.001935; origin xyz=-0.008681 -0.034681 0.005931 rpy=0 0 0 -> xyz=-0.00869 -0.034684 0.005904 rpy=0 0 0
- joint Revolute_30: axis 0.49842 -0.866934 0.001748 -> 0.498367 -0.866964 0.001935; origin xyz=-0.007038 -0.033771 -0.011104 rpy=0 0 0 -> xyz=-0.007051 -0.03378 -0.011069 rpy=0 0 0
- joint Revolute_31: axis 0.501578 0.865112 -0.000872 -> 0.501629 0.865083 0.000253; origin xyz=-0.008528 0.034703 -0.006021 rpy=0 0 0 -> xyz=-0.008516 0.034706 -0.006025 rpy=0 0 0
- joint Revolute_32: axis 0.501578 0.865112 -0.000872 -> 0.501629 0.865083 0.000253; origin xyz=-0.006966 0.033815 0.011015 rpy=0 0 0 -> xyz=-0.007012 0.033829 0.010943 rpy=0 0 0
- joint Revolute_33: axis -0.001566 -0.972184 -0.234213 -> -0.001325 -0.972931 -0.231091; origin xyz=-0.015045 0.016136 0.042 rpy=0 0 0 -> xyz=-0.015064 0.016268 0.041942 rpy=0 0 0
- joint Revolute_34: axis 0.999998 -0.001822 0.000875 -> 0.999996 -0.001881 0.002188; origin xyz=0.02571 -0.024838 -0.00595 rpy=0 0 0 -> xyz=0.025716 -0.024858 -0.005837 rpy=0 0 0
- joint Revolute_35: axis -0.002021 -0.900818 0.434191 -> -0.002645 -0.900636 0.434566; origin xyz=-3.4e-05 0.040341 0.024966 rpy=0 0 0 -> xyz=-8.3e-05 0.040352 0.024949 rpy=0 0 0
- joint Revolute_36: axis -0.999998 0.001822 -0.000875 -> -0.999996 0.001881 -0.002188; origin xyz=-0.025801 -0.022923 0.011049 rpy=0 0 0 -> xyz=-0.025817 -0.022918 0.011025 rpy=0 0 0
- joint Revolute_7: axis 0.0 0.971958 0.235153 -> 0.0 0.972693 0.232097; origin xyz=-0.0255 0.025028 0.006055 rpy=0 0 0 -> xyz=-0.0255 0.025047 0.005976 rpy=0 0 0
- joint Revolute_8: axis -0.0 -0.902007 0.431722 -> -0.0 -0.902181 0.431357; origin xyz=-0.0255 -0.023227 0.011116 rpy=0 0 0 -> xyz=-0.0255 -0.023231 0.011107 rpy=0 0 0
- joint Revolute_9: axis 0.781728 -0.451331 -0.430351 -> 0.783126 -0.452138 -0.426948; origin xyz=0.03288 0.010462 -0.011082 rpy=0 0 0 -> xyz=0.032916 0.010441 -0.010994 rpy=0 0 0
- joint Rigid_59: origin xyz=-0.012869 0.022384 0.039711 rpy=0 0 0 -> xyz=-0.01292 0.022363 0.039706 rpy=0 0 0
- joint Rigid_60: origin xyz=0.025715 1.3e-05 0.039778 rpy=0 0 0 -> xyz=0.025663 -1e-05 0.039812 rpy=0 0 0
- joint Rigid_61: origin xyz=-0.025785 0.000107 0.039733 rpy=0 0 0 -> xyz=-0.025836 8.7e-05 0.039699 rpy=0 0 0
- joint Rigid_62: origin xyz=-0.012951 -0.022217 0.039778 rpy=0 0 0 -> xyz=-0.013004 -0.022237 0.039749 rpy=0 0 0
- joint Rigid_63: origin xyz=-0.01295 -0.022216 0.039778 rpy=0 0 0 -> xyz=-0.013004 -0.022237 0.039749 rpy=0 0 0
- joint Rigid_64: origin xyz=-0.01287 0.022386 0.04071 rpy=0 0 0 -> xyz=-0.012922 0.022364 0.040706 rpy=0 0 0
- joint Rigid_65: origin xyz=-1e-06 1e-06 0.001 rpy=0 0 0 -> xyz=-3e-06 1e-06 0.001 rpy=0 0 0
- joint Rigid_66: origin xyz=-1e-06 2e-06 0.001 rpy=0 0 0 -> xyz=-2e-06 1e-06 0.001 rpy=0 0 0
- joint Rigid_67: origin xyz=-0.085 0.000155 -7.4e-05 rpy=0 0 0 -> xyz=-0.084999 0.00016 -0.000186 rpy=0 0 0
- joint Rigid_68: origin xyz=-0.232158 0.256117 -0.00059 rpy=0 0 0 -> xyz=-0.232142 0.256131 -0.000757 rpy=0 0 0
- joint Rigid_69: origin xyz=-0.189524 0.329651 -0.000664 rpy=0 0 0 -> xyz=-0.189504 0.329663 -0.000736 rpy=0 0 0
- joint Rigid_70: origin xyz=0.105725 0.329113 -0.000406 rpy=0 0 0 -> xyz=0.105745 0.329108 -9e-05 rpy=0 0 0
- joint Rigid_71: origin xyz=0.148091 0.255424 -0.000257 rpy=0 0 0 -> xyz=0.148106 0.255416 7.5e-05 rpy=0 0 0
- joint Rigid_77: origin xyz=-0.042142 0.195074 -0.002332 rpy=0 0 0 -> xyz=-0.042128 0.195078 -0.002282 rpy=0 0 0
- joint Slider_13: axis 0.371624 -0.217029 0.902659 -> 0.369151 -0.214507 0.904276; origin xyz=0.069062 -0.040466 0.227725 rpy=0 0 0 -> xyz=0.068432 -0.03984 0.228025 rpy=0 0 0
- joint Slider_14: axis -0.002141 0.434195 0.900816 -> -0.00375 0.434573 0.900629; origin xyz=-0.022183 0.11672 0.21012 rpy=0 0 0 -> xyz=-0.02256 0.116805 0.210031 rpy=0 0 0
- joint Slider_15: axis -0.377094 -0.216348 0.900552 -> -0.377381 -0.213518 0.901107; origin xyz=-0.110587 -0.06352 0.204943 rpy=0 0 0 -> xyz=-0.110669 -0.062847 0.205106 rpy=0 0 0
- joint Slider_16: axis 0.373767 -0.218269 0.901475 -> 0.370839 -0.215482 0.903353; origin xyz=0.068012 -0.064911 0.222322 rpy=0 0 0 -> xyz=0.0673 -0.064247 0.22273 rpy=0 0 0
- joint Slider_17: axis -0.002144 0.431721 0.902005 -> -0.003749 0.431354 0.902175; origin xyz=-0.000515 0.126842 0.20537 rpy=0 0 0 -> xyz=-0.0009 0.126758 0.20542 rpy=0 0 0
- joint Slider_18: axis -0.379236 -0.217587 0.899353 -> -0.379485 -0.214736 0.899933; origin xyz=-0.091019 -0.07725 0.209794 rpy=0 0 0 -> xyz=-0.091079 -0.076585 0.210013 rpy=0 0 0
